Commit message: marrtinox

File: urdf/marrtinox.urdf.xacro (robot description, xacro)
@@ -49,5 +49,5 @@
             <geometry>
                 <!--<box size="${b_length} ${b_width} ${b_height}"/>-->
-                <mesh filename="package://marrtino_utilities/urdf/marrtinox/base.dae" scale="0.001 0.001 0.001" />
+                <mesh filename="package://marrtinox_description/urdf/marrtinox/base.dae" scale="0.001 0.001 0.001" />
             </geometry>
         </visual>
